File: FullProject/final_project/_autosave-final_project.kicad_pcb (KiCad board)
At the start: 2 copper layers, 46 parts, among them J1 Conn_WallSocket, J2 Weight Sensor Connector, J3 PIR Array Connector 01, J4 PIR Array Connector 02, J5 PIR Array Connector 03, J6 pH Sensor Connector, J7 Keypad Connector, J8 LCD Connector, J9 Conn_01x02_Female, M1 Motor_DC, M2 Motor_Servo, Q1 2N4403, U1 L7805, U2 LM7809_TO220, U3 LM7812_TO220, U4 ATmega32A-P, U5 L293D, U6 SIM900, U7 DS3232M, U8 PCF8574

Commit message: add
Parts:
- C1, C2, C3: footprint Capacitor_SMD:C_0201_0603Metric -> Capacitor_THT:CP_Axial_L10.0mm_D4.5mm_P15.00mm_Horizontal
- C4: footprint Crystal:Crystal_AT310_D3.0mm_L10.0mm_Vertical -> Capacitor_THT:CP_Axial_L11.0mm_D6.0mm_P18.00mm_Horizontal
- C5: footprint Capacitor_SMD:C_0201_0603Metric -> Capacitor_THT:CP_Axial_L11.0mm_D5.0mm_P18.00mm_Horizontal
- J9: footprint Crystal:Crystal_C38-LF_D3.0mm_L8.0mm_Vertical -> Connector_Phoenix_MSTB:PhoenixContact_MSTBA_2,5_2-G_1x02_P5.00mm_Horizontal
- R5, R6, R7, R8: footprint Resistor_THT:R_Axial_DIN0411_L9.9mm_D3.6mm_P20.32mm_Horizontal -> Resistor_THT:R_Axial_DIN0207_L6.3mm_D2.5mm_P7.62mm_Horizontal
- Temperature1: footprint Package_TO_SOT_THT:TO-92_Inline -> Connector_PinSocket_2.54mm:PinSocket_1x03_P2.54mm_Vertical
- Ultrasonic1: value Ultrasonic Connector -> Conn_01x04_Female; footprint Connector_PinHeader_2.00mm:PinHeader_1x04_P2.00mm_Vertical -> Connector_PinSocket_2.54mm:PinSocket_1x04_P2.54mm_Vertical
- moved D5 184.3 mm to (250.9, 21.7)
- moved J9 171.8 mm to (43.9, 180.9), turned to -90 degrees
- moved Q1 151.4 mm to (45.5, 26.5), turned to -90 degrees
- moved C6 142.5 mm to (223.9, 88.6), turned to 90 degrees
- moved R8 128.1 mm to (221.1, 146.2), turned to 90 degrees
- moved Temperature1 124.8 mm to (136.8, 15.9), turned to 90 degrees
- moved C3 119.5 mm to (25.9, 20.8)
- moved R7 119.3 mm to (211.4, 146.8), turned to 90 degrees
- moved R2 112.8 mm to (45.7, 50.9), turned to -90 degrees
- moved L1 110.2 mm to (187.1, 88.8)
- moved R1 108.2 mm to (45.6, 38.7), turned to -90 degrees
- moved R3 104.7 mm to (88.5, 34.5)
- moved U8 99.9 mm to (245.2, 89.0)
- moved R6 93.7 mm to (177.1, 134.5), turned to 90 degrees
- moved R5 91.2 mm to (187.2, 134.7), turned to 90 degrees
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Routing:
- net Net-(BZ1-Pad2): track 0.00 -> 214.2 mm
- net Net-(C4-Pad1): track 0.00 -> 110.5 mm
- net Net-(D1-Pad1): track 0.00 -> 39.8 mm
- net Net-(D2-Pad1): track 0.00 -> 39.7 mm
- net Net-(M2-Pad2): track 0.00 -> 24.2 mm
