File: FullProject/final_project/_autosave-final_project.kicad_sch (KiCad schematic)
At the start: 46 parts, among them J1 Conn_WallSocket, J2 Weight Sensor Connector, J3 PIR Array Connector 01, J4 PIR Array Connector 02, J5 PIR Array Connector 03, J6 pH Sensor Connector, J7 Keypad Connector, J8 LCD Connector, J9 Conn_01x02_Female, M1 Motor_DC, M2 Motor_Servo, Q1 2N4403, U1 L7805, U2 LM7809_TO220, U3 LM7812_TO220, U4 ATmega32A-P, U5 L293D, U6 SIM900, U7 DS3232M, U8 PCF8574

Commit message: add
Parts:
- C1, C2: footprint Capacitor_THT:CP_Axial_L11.0mm_D5.0mm_P18.00mm_Horizontal -> Capacitor_THT:CP_Axial_L10.0mm_D4.5mm_P15.00mm_Horizontal
- C3: footprint Capacitor_SMD:C_0201_0603Metric -> Capacitor_THT:CP_Axial_L10.0mm_D4.5mm_P15.00mm_Horizontal
- C5: footprint Capacitor_SMD:C_0201_0603Metric -> Capacitor_THT:CP_Axial_L11.0mm_D5.0mm_P18.00mm_Horizontal
- J9: footprint Crystal:Crystal_C38-LF_D3.0mm_L8.0mm_Vertical -> Connector_Phoenix_MSTB:PhoenixContact_MSTBA_2,5_2-G_1x02_P5.00mm_Horizontal
- R5, R6, R7, R8: footprint Resistor_THT:R_Axial_DIN0411_L9.9mm_D3.6mm_P20.32mm_Horizontal -> Resistor_THT:R_Axial_DIN0207_L6.3mm_D2.5mm_P7.62mm_Horizontal
- Temperature1: footprint Package_TO_SOT_THT:TO-92_Inline -> Connector_PinSocket_2.54mm:PinSocket_1x03_P2.54mm_Vertical
- Ultrasonic1: footprint Connector_PinHeader_2.00mm:PinHeader_1x04_P2.00mm_Vertical -> Connector_PinSocket_2.54mm:PinSocket_1x04_P2.54mm_Vertical
Changed lines of the file:
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@@
       (effects (font (size 1.27 1.27)) (justify left))
     )
-    (property "Footprint" "Resistor_THT:R_Axial_DIN0411_L9.9mm_D3.6mm_P20.32mm_Horizontal" (id 2) (at 327.152 146.05 90)
+    (property "Footprint" "Resistor_THT:R_Axial_DIN0207_L6.3mm_D2.5mm_P7.62mm_Horizontal" (id 2) (at 327.152 146.05 90)
       (effects (font (size 1.27 1.27)) hide)
     )
@@
       (effects (font (size 1.27 1.27)) (justify left))
     )
-    (property "Footprint" "Connector_PinHeader_2.00mm:PinHeader_1x04_P2.00mm_Vertical" (id 2) (at 262.89 36.83 0)
+    (property "Footprint" "Connector_PinSocket_2.54mm:PinSocket_1x04_P2.54mm_Vertical" (id 2) (at 262.89 36.83 0)
       (effects (font (size 1.27 1.27)) hide)
     )
@@
       (effects (font (size 1.27 1.27)) (justify right))
     )
-    (property "Footprint" "Package_TO_SOT_THT:TO-92_Inline" (id 2) (at 181.61 46.99 0)
+    (property "Footprint" "Connector_PinSocket_2.54mm:PinSocket_1x03_P2.54mm_Vertical" (id 2) (at 181.61 46.99 0)
       (effects (font (size 1.27 1.27)) hide)
     )
@@
       (effects (font (size 1.27 1.27)) (justify left))
     )
-    (property "Footprint" "Resistor_THT:R_Axial_DIN0411_L9.9mm_D3.6mm_P20.32mm_Horizontal" (id 2) (at 285.242 138.43 90)
+    (property "Footprint" "Resistor_THT:R_Axial_DIN0207_L6.3mm_D2.5mm_P7.62mm_Horizontal" (id 2) (at 285.242 138.43 90)
       (effects (font (size 1.27 1.27)) hide)
     )
@@
       (effects (font (size 1.27 1.27)) (justify left))
     )
-    (property "Footprint" "Capacitor_THT:CP_Axial_L11.0mm_D5.0mm_P18.00mm_Horizontal" (id 2) (at 40.3352 83.82 0)
+    (property "Footprint" "Capacitor_THT:CP_Axial_L10.0mm_D4.5mm_P15.00mm_Horizontal" (id 2) (at 40.3352 83.82 0)
       (effects (font (size 1.27 1.27)) hide)
     )
@@
     (property "Reference" "J9" (id 0) (at 56.515 254 0))
     (property "Value" "Conn_01x02_Female" (id 1) (at 56.515 256.54 0))
-    (property "Footprint" "Crystal:Crystal_C38-LF_D3.0mm_L8.0mm_Vertical" (id 2) (at 55.88 261.62 0)
+    (property "Footprint" "Connector_Phoenix_MSTB:PhoenixContact_MSTBA_2,5_2-G_1x02_P5.00mm_Horizontal" (id 2) (at 55.88 261.62 0)
       (effects (font (size 1.27 1.27)) hide)
     )
@@
     (property "Reference" "C3" (id 0) (at 58.42 35.56 90))
     (property "Value" "10 μF" (id 1) (at 58.42 38.1 90))
-    (property "Footprint" "Capacitor_SMD:C_0201_0603Metric" (id 2) (at 54.61 44.1452 0)
+    (property "Footprint" "Capacitor_THT:CP_Axial_L10.0mm_D4.5mm_P15.00mm_Horizontal" (id 2) (at 54.61 44.1452 0)
       (effects (font (size 1.27 1.27)) hide)
     )
@@
       (effects (font (size 1.27 1.27)) (justify left))
     )
-    (property "Footprint" "Resistor_THT:R_Axial_DIN0411_L9.9mm_D3.6mm_P20.32mm_Horizontal" (id 2) (at 332.232 146.05 90)
+    (property "Footprint" "Resistor_THT:R_Axial_DIN0207_L6.3mm_D2.5mm_P7.62mm_Horizontal" (id 2) (at 332.232 146.05 90)
       (effects (font (size 1.27 1.27)) hide)
     )
@@
       (effects (font (size 1.27 1.27)) (justify left))
     )
-    (property "Footprint" "Capacitor_SMD:C_0201_0603Metric" (id 2) (at 159.7152 91.44 0)
+    (property "Footprint" "Capacitor_THT:CP_Axial_L11.0mm_D5.0mm_P18.00mm_Horizontal" (id 2) (at 159.7152 91.44 0)
       (effects (font (size 1.27 1.27)) hide)
     )
@@
       (effects (font (size 1.27 1.27)) (justify left))
     )
-    (property "Footprint" "Capacitor_THT:CP_Axial_L11.0mm_D5.0mm_P18.00mm_Horizontal" (id 2) (at 40.3352 107.95 0)
+    (property "Footprint" "Capacitor_THT:CP_Axial_L10.0mm_D4.5mm_P15.00mm_Horizontal" (id 2) (at 40.3352 107.95 0)
       (effects (font (size 1.27 1.27)) hide)
     )
@@
       (effects (font (size 1.27 1.27)) (justify left))
     )
-    (property "Footprint" "Resistor_THT:R_Axial_DIN0411_L9.9mm_D3.6mm_P20.32mm_Horizontal" (id 2) (at 290.322 138.43 90)
+    (property "Footprint" "Resistor_THT:R_Axial_DIN0207_L6.3mm_D2.5mm_P7.62mm_Horizontal" (id 2) (at 290.322 138.43 90)
       (effects (font (size 1.27 1.27)) hide)
     )
@@
     )
     (path "/66e3520f-603c-4ad5-982c-42f96186bda7"
-      (reference "C1") (unit 1) (value "10 μF") (footprint "Capacitor_THT:CP_Axial_L11.0mm_D5.0mm_P18.00mm_Horizontal")
+      (reference "C1") (unit 1) (value "10 μF") (footprint "Capacitor_THT:CP_Axial_L10.0mm_D4.5mm_P15.00mm_Horizontal")
     )
     (path "/edf4054d-41a8-49a4-a0bf-064d4fae46db"
-      (reference "C2") (unit 1) (value "0.1 μF") (footprint "Capacitor_THT:CP_Axial_L11.0mm_D5.0mm_P18.00mm_Horizontal")
+      (reference "C2") (unit 1) (value "0.1 μF") (footprint "Capacitor_THT:CP_Axial_L10.0mm_D4.5mm_P15.00mm_Horizontal")
     )
     (path "/bf7daf89-d534-4fdf-be92-a7010336efdd"
-      (reference "C3") (unit 1) (value "10 μF") (footprint "Capacitor_SMD:C_0201_0603Metric")
+      (reference "C3") (unit 1) (value "10 μF") (footprint "Capacitor_THT:CP_Axial_L10.0mm_D4.5mm_P15.00mm_Horizontal")
     )
     (path "/60c6b86e-0c1d-47cb-ab4d-2cb37ff961b5"
@@
     )
     (path "/dde8240f-5c2e-40a9-a46a-d9fc31bd2aac"
-      (reference "C5") (unit 1) (value "0.1 μF") (footprint "Capacitor_SMD:C_0201_0603Metric")
+      (reference "C5") (unit 1) (value "0.1 μF") (footprint "Capacitor_THT:CP_Axial_L11.0mm_D5.0mm_P18.00mm_Horizontal")
     )
     (path "/6a5c3930-a0dd-4739-a00a-10ae4b32ea4a"
@@
     )
     (path "/9349c33e-82e3-4b38-8a69-2cf2953d5b3a"
-      (reference "J9") (unit 1) (value "Conn_01x02_Female") (footprint "Crystal:Crystal_C38-LF_D3.0mm_L8.0mm_Vertical")
+      (reference "J9") (unit 1) (value "Conn_01x02_Female") (footprint "Connector_Phoenix_MSTB:PhoenixContact_MSTBA_2,5_2-G_1x02_P5.00mm_Horizontal")
     )
     (path "/0c9bf32b-4a6c-4391-8a56-38b7d9d09a1c"
@@
     )
     (path "/57f5177e-7a5a-45b5-bff8-dcd0c819d009"
-      (reference "R5") (unit 1) (value "R") (footprint "Resistor_THT:R_Axial_DIN0411_L9.9mm_D3.6mm_P20.32mm_Horizontal")
+      (reference "R5") (unit 1) (value "R") (footprint "Resistor_THT:R_Axial_DIN0207_L6.3mm_D2.5mm_P7.62mm_Horizontal")
     )
     (path "/f2f89f62-62cf-4904-ae39-aa2de3fbe8ef"
-      (reference "R6") (unit 1) (value "R") (footprint "Resistor_THT:R_Axial_DIN0411_L9.9mm_D3.6mm_P20.32mm_Horizontal")
+      (reference "R6") (unit 1) (value "R") (footprint "Resistor_THT:R_Axial_DIN0207_L6.3mm_D2.5mm_P7.62mm_Horizontal")
     )
     (path "/197c478e-16cc-4799-9b49-8d61b9af7099"
-      (reference "R7") (unit 1) (value "R") (footprint "Resistor_THT:R_Axial_DIN0411_L9.9mm_D3.6mm_P20.32mm_Horizontal")
+      (reference "R7") (unit 1) (value "R") (footprint "Resistor_THT:R_Axial_DIN0207_L6.3mm_D2.5mm_P7.62mm_Horizontal")
     )
     (path "/c208471a-71a7-45af-bee0-3c959e07ed36"
-      (reference "R8") (unit 1) (value "R") (footprint "Resistor_THT:R_Axial_DIN0411_L9.9mm_D3.6mm_P20.32mm_Horizontal")
+      (reference "R8") (unit 1) (value "R") (footprint "Resistor_THT:R_Axial_DIN0207_L6.3mm_D2.5mm_P7.62mm_Horizontal")
     )
     (path "/0b89cc82-93fc-4844-a02d-d043f0af0213"
@@
     )
     (path "/2ca04f4d-2338-4692-a827-24a5eb302c79"
-      (reference "Temperature1") (unit 1) (value "DS18B20") (footprint "Package_TO_SOT_THT:TO-92_Inline")
+      (reference "Temperature1") (unit 1) (value "DS18B20") (footprint "Connector_PinSocket_2.54mm:PinSocket_1x03_P2.54mm_Vertical")
     )
     (path "/9e9b4019-8c24-40fb-a71e-88e462492108"
@@
     )
     (path "/1f68107a-7269-4116-9c75-1e34c456d541"
-      (reference "Ultrasonic1") (unit 1) (value "Conn_01x04_Female") (footprint "Connector_PinHeader_2.00mm:PinHeader_1x04_P2.00mm_Vertical")
-    )
-  )
+      (reference "Ultrasonic1") (unit 1) (value "Conn_01x04_Female") (footprint "Connector_PinSocket_2.54mm:PinSocket_1x04_P2.54mm_Vertical")
+    )
+  )
