File: FullProject/final_project/final_project.kicad_pcb (KiCad board)
At the start: 2 copper layers, 46 parts, among them J1 Conn_WallSocket, J2 Weight Sensor Connector, J3 PIR Array Connector 01, J4 PIR Array Connector 02, J5 PIR Array Connector 03, J6 pH Sensor Connector, J7 Keypad Connector, J8 LCD Connector, J9 Conn_01x02_Female, M1 Motor_DC, M2 Motor_Servo, Q1 2N4403, U1 L7805, U2 LM7809_TO220, U3 LM7812_TO220, U4 ATmega32A-P, U5 L293D, U6 SIM900, U7 DS3232M, U8 PCF8574

Commit message: add
Parts:
- C1, C2, C3: footprint Capacitor_SMD:C_0201_0603Metric -> Capacitor_THT:CP_Axial_L10.0mm_D4.5mm_P15.00mm_Horizontal
- C4: footprint Crystal:Crystal_AT310_D3.0mm_L10.0mm_Vertical -> Capacitor_THT:CP_Axial_L11.0mm_D6.0mm_P18.00mm_Horizontal
- C5: footprint Capacitor_SMD:C_0201_0603Metric -> Capacitor_THT:CP_Axial_L11.0mm_D5.0mm_P18.00mm_Horizontal
- J9: footprint Crystal:Crystal_C38-LF_D3.0mm_L8.0mm_Vertical -> Connector_Phoenix_MSTB:PhoenixContact_MSTBA_2,5_2-G_1x02_P5.00mm_Horizontal
- R5, R6, R7, R8: footprint Resistor_THT:R_Axial_DIN0411_L9.9mm_D3.6mm_P20.32mm_Horizontal -> Resistor_THT:R_Axial_DIN0207_L6.3mm_D2.5mm_P7.62mm_Horizontal
- RL1, RL2: moved to B.Cu
- Temperature1: footprint Package_TO_SOT_THT:TO-92_Inline -> Connector_PinSocket_2.54mm:PinSocket_1x03_P2.54mm_Vertical
- Ultrasonic1: value Ultrasonic Connector -> Conn_01x04_Female; footprint Connector_PinHeader_2.00mm:PinHeader_1x04_P2.00mm_Vertical -> Connector_PinSocket_2.54mm:PinSocket_1x04_P2.54mm_Vertical
- moved D5 184.3 mm to (250.9, 21.7)
- moved J9 171.8 mm to (43.9, 180.9), turned to -90 degrees
- moved Q1 151.4 mm to (45.5, 26.5), turned to -90 degrees
- moved C6 142.5 mm to (223.9, 88.6), turned to 90 degrees
- moved R8 128.1 mm to (221.1, 146.2), turned to 90 degrees
- moved Temperature1 124.8 mm to (136.8, 15.9), turned to 90 degrees
- moved C3 119.5 mm to (25.9, 20.8)
- moved R7 119.3 mm to (211.4, 146.8), turned to 90 degrees
- moved R2 112.8 mm to (45.7, 50.9), turned to -90 degrees
- moved L1 110.2 mm to (187.1, 88.8)
- moved R1 108.2 mm to (45.6, 38.7), turned to -90 degrees
- moved R3 104.7 mm to (88.5, 34.5)
- moved U8 99.9 mm to (245.2, 89.0)
- moved R6 93.7 mm to (177.1, 134.5), turned to 90 degrees
- moved R5 91.2 mm to (187.2, 134.7), turned to 90 degrees
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Routing:
- net Net-(BZ1-Pad2): track 0.00 -> 523.9 mm
- net Net-(M2-Pad2): track 0.00 -> 130.7 mm
- net Net-(C4-Pad1): track 0.00 -> 110.5 mm
- net Net-(D1-Pad1): track 0.00 -> 39.8 mm
- net Net-(D2-Pad1): track 0.00 -> 39.7 mm
- net Net-(M1-Pad2): track 0.00 -> 33.4 mm
- net Net-(C3-Pad1): track 0.00 -> 28.7 mm
- net Net-(M1-Pad1): track 0.00 -> 16.0 mm

Commit message: add
Parts:
- removed U6: SIM900, RF_GSM:SIMCom_SIM900
- added J10: Conn_01x03_Female, Connector_PinSocket_2.54mm:PinSocket_1x03_P2.54mm_Vertical, F.Cu at (111.2, 126.2)
- moved J8 33.9 mm to (279.1, 115.1), turned to 180 degrees
- moved R7 7.85 mm to (212.8, 139.1), turned to -90 degrees
- moved R8 7.32 mm to (221.3, 138.9), turned to -90 degrees
- moved RL1 2.23 mm to (259.6, 135.9)
- moved D5 2.05 mm to (252.9, 21.8)
- turned R5 to -90 degrees
- turned R6 to -90 degrees
Routing:
- net Net-(C3-Pad1): track 28.7 -> 553.8 mm
- net Net-(BZ1-Pad2): track 523.9 -> 1032.8 mm, vias 0 -> 1
- net Net-(J6-Pad3): track 0.00 -> 154.5 mm
- net Net-(J8-Pad4): track 0.00 -> 75.8 mm
- net Net-(J8-Pad5): track 0.00 -> 75.1 mm
- net Net-(J8-Pad6): track 0.00 -> 72.6 mm
- net Net-(C6-Pad1): track 0.00 -> 55.7 mm
- net Net-(J8-Pad14): track 0.00 -> 32.0 mm
- net Net-(J8-Pad13): track 0.00 -> 31.2 mm
- net Net-(J8-Pad11): track 0.00 -> 30.7 mm
- net Net-(J8-Pad12): track 0.00 -> 30.4 mm
- net Net-(BZ1-Pad1): track 0.00 -> 26.6 mm

Commit message: add
Connections:
- J5 pad 2: Net-(C3-Pad1) -> Net-(J5-Pad2)
- U4 pad 36: Net-(C3-Pad1) -> Net-(J5-Pad2)
Routing:
- net Net-(C3-Pad1): track 553.8 -> 682.5 mm

Commit message: add
Parts:
- moved C2 23.0 mm to (27.9, 58.0), turned to -90 degrees
- moved C1 21.0 mm to (27.7, 34.0), turned to -90 degrees
- moved C3 14.7 mm to (40.5, 19.1), turned to 180 degrees
- moved Q1 2.66 mm to (48.1, 25.9)
- moved R2 2.57 mm to (48.2, 50.6)
- moved R1 2.53 mm to (48.1, 39.1)
- moved HX1 0.55 mm to (61.9, 21.0)
Routing:
- net Net-(BZ1-Pad2): track 1032.8 -> 1268.2 mm, vias 1 -> 2
- net Net-(C1-Pad1): track 0.00 -> 189.5 mm
- net Net-(C6-Pad1): track 55.7 -> 170.9 mm
- net Net-(C3-Pad1): track 682.5 -> 788.8 mm
- net Net-(C2-Pad2): track 0.00 -> 68.0 mm
- net Net-(C5-Pad2): track 0.00 -> 51.2 mm
- net Net-(HX1-Pad8): track 0.00 -> 41.1 mm, vias 0 -> 1
- net Net-(HX1-Pad7): track 0.00 -> 39.3 mm
- net Net-(C5-Pad1): track 0.00 -> 29.4 mm
- net Net-(HX1-Pad4): track 0.00 -> 29.2 mm
- net Net-(Q1-Pad3): track 0.00 -> 10.6 mm
- net Net-(HX1-Pad2): track 0.00 -> 8.73 mm

Commit message: add
Parts:
- moved J7 210.7 mm to (32.5, 88.8), turned to 0 degrees
Routing:
- net Net-(R6-Pad1): track 0.00 -> 215.4 mm, vias 0 -> 2
- net Net-(RL2-PadA1): track 0.00 -> 209.6 mm, vias 0 -> 2
- net Net-(R5-Pad1): track 0.00 -> 187.2 mm, vias 0 -> 2
- net Net-(U4-Pad16): track 0.00 -> 177.8 mm, vias 0 -> 1
- net Net-(U4-Pad17): track 0.00 -> 165.6 mm, vias 0 -> 1
- net Net-(BZ1-Pad1): track 26.6 -> 190.2 mm, vias 0 -> 1
- net Net-(RL1-PadA1): track 0.00 -> 148.7 mm, vias 0 -> 2
- net Net-(J4-Pad2): track 0.00 -> 138.8 mm, vias 0 -> 1
- net Net-(J5-Pad2): track 0.00 -> 136.4 mm, vias 0 -> 1
- net Net-(J7-Pad8): track 0.00 -> 133.6 mm, vias 0 -> 2
- net Net-(HX1-Pad11): track 0.00 -> 132.7 mm, vias 0 -> 2
- net Net-(HX1-Pad12): track 0.00 -> 132.1 mm, vias 0 -> 2
- net Net-(J7-Pad7): track 0.00 -> 128.6 mm, vias 0 -> 2
- net Net-(J7-Pad6): track 0.00 -> 122.7 mm, vias 0 -> 2
- net Net-(J7-Pad5): track 0.00 -> 116.4 mm, vias 0 -> 2
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Other:
- copper layers 2 -> 4

Commit message: add
Parts:
- added J11: Conn_WallSocket, Connector_AMASS:AMASS_XT60-M_1x02_P7.20mm_Vertical, F.Cu at (281.0, 140.0)
- added J12: Conn_WallSocket, Connector_AMASS:AMASS_XT60-M_1x02_P7.20mm_Vertical, F.Cu at (280.0, 160.0)
- J10: value Conn_01x03_Female -> SIM 900D Connector
- RL1, RL2: moved to F.Cu
- moved J7 25.3 mm to (24.8, 112.9), turned to 180 degrees
- moved RL1 11.5 mm to (271.1, 135.0), turned to 180 degrees
- moved RL2 11.3 mm to (271.1, 156.0), turned to 180 degrees
- moved Temperature1 5.50 mm to (136.8, 21.4)
- moved J2 4.98 mm to (110.6, 20.5)
- moved J4 3.61 mm to (201.9, 19.7)
- moved J3 3.50 mm to (181.1, 19.6)
- moved J5 3.42 mm to (223.4, 19.5)
- moved Ultrasonic1 3.10 mm to (159.1, 19.1)
Connections:
- RL1 pad 11: unconnected-(RL1-Pad11) -> Net-(RL1-Pad11)
- RL1 pad 12: unconnected-(RL1-Pad12) -> Net-(RL1-Pad12)
- RL2 pad 11: unconnected-(RL2-Pad11) -> Net-(RL2-Pad11)
- RL2 pad 12: unconnected-(RL2-Pad12) -> Net-(RL2-Pad12)
Routing:
- net Net-(J3-Pad2): track 88.5 -> 314.7 mm, vias 1 -> 5
- net Net-(J4-Pad2): track 138.8 -> 302.0 mm, vias 1 -> 5
- net Net-(J5-Pad2): track 136.4 -> 283.6 mm, vias 1 -> 5
- net Net-(Temperature1-Pad2): track 60.0 -> 158.6 mm, vias 1 -> 6
- net Net-(BZ1-Pad1): track 190.2 -> 267.5 mm, vias 1 -> 4
- net Net-(J7-Pad1): track 107.4 -> 159.9 mm
- net Net-(U4-Pad17): track 165.6 -> 212.5 mm
- net Net-(J7-Pad2): track 107.5 -> 153.4 mm
- net Net-(U4-Pad16): track 177.8 -> 218.6 mm, vias 1 -> 3
- net Net-(R5-Pad1): track 187.2 -> 227.6 mm
- net Net-(J7-Pad3): track 107.4 -> 145.9 mm
- net Net-(J7-Pad4): track 106.8 -> 138.1 mm
- net Net-(RL1-Pad12): track 0.00 -> 26.7 mm
- net Net-(RL2-Pad12): track 0.00 -> 24.8 mm
- net Net-(J7-Pad5): track 116.4 -> 131.8 mm, vias 2 -> 1
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- added copper zone on B.Cu, net Net-(C3-Pad1)
- added copper zone on F.Cu, net Net-(C3-Pad1)
Other:
- copper layers 4 -> 2
- board text added: "SIM 900D"

Commit message: add
Parts:
- removed J1: Conn_WallSocket, Connector_AMASS:AMASS_XT60-M_1x02_P7.20mm_Vertical
- J11: value Conn_WallSocket -> Lamp Connector
- J12: value Conn_WallSocket -> Padding Wheel Connector
- J9: value Conn_01x02_Female -> 12V AC SUPPLY
- M2: value Motor_Servo -> Servo Motor Connector
- R5, R6, R7, R8: value R -> 10K
- RL1: value FINDER-36.11 -> Lamp Control Relay
- RL2: value FINDER-36.11 -> Padding Wheel Control Relay
- U4: value ATmega32A-P -> ATmega32
- U5: value L293D -> L293D Motor Controller
- U7: value DS3232M -> DS3232M RTC
- U8: value PCF8574 -> PCF8574 I2C to 8bit
- Ultrasonic1: value Conn_01x04_Female -> Ultrasonic Connector
- moved Ultrasonic1 0.90 mm to (159.1, 20.0)
Routing:
- net Net-(M2-Pad2): track 130.7 -> 154.4 mm
- net Net-(C3-Pad1): track 869.5 -> 857.0 mm
- net Net-(BZ1-Pad2): track 1325.6 -> 1336.3 mm
- net Net-(U4-Pad17): track 212.5 -> 213.4 mm
- net Net-(U4-Pad16): track 218.6 -> 219.5 mm
Other:
- board text added: "+"
- board text added: "+12V"
- board text added: "+5V"
- board text added: "-"
- board text added: "D0"
- board text added: "ECHO"
- board text added: "GND"
- board text added: "OUT"
- board text added: "RXD"
- board text added: "Signal"
- board text added: "TR"
- board text added: "TXD"
- board text added: "Temp"
- board text added: "VCC"

Commit message: ADD
Parts:
- C4: value C_Polarized -> 470μF
- C6: value C_Polarized -> 10000μF
- L1: value INDUCTOR -> 27uH
- U2: value LM7809_TO220 -> LM7809
- U3: value LM7812_TO220 -> LM7812
- moved Temperature1 2.00 mm to (136.8, 19.4)
Routing:
- net Net-(C3-Pad1): track 857.0 -> 898.7 mm
- net Net-(Temperature1-Pad2): track 158.6 -> 160.6 mm
- net Net-(J8-Pad4): track 75.8 -> 77.4 mm
- net Net-(M2-Pad1): track 75.8 -> 74.5 mm
- net Net-(U4-Pad16): track 219.5 -> 218.6 mm
- net Net-(J8-Pad6): track 72.6 -> 73.1 mm
Other:
- board text added: "D4"
- board text added: "D5"
- board text added: "D6"
- board text added: "D7"
- board text added: "E"
- board text added: "RS"
- board text added: "RW"
- board text added: "VDD"
