File: FullProject/final_project/final_project.kicad_pcb (KiCad board)
At the start: 2 copper layers, 47 parts, among them J10 SIM 900D Connector, J11 Lamp Connector, J12 Padding Wheel Connector, J2 Weight Sensor Connector, J3 PIR Array Connector 01, J4 PIR Array Connector 02, J5 PIR Array Connector 03, J6 pH Sensor Connector, J7 Keypad Connector, J8 LCD Connector, J9 12V AC SUPPLY, M1 Motor_DC, M2 Servo Motor Connector, Q1 2N4403, U1 L7805, U2 LM7809, U3 LM7812, U4 ATmega32, U5 L293D Motor Controller, U7 DS3232M RTC, U8 PCF8574 I2C to 8bit

Commit message: add
Parts:
- added REF**: MountingHole_4.3mm_M4_Pad, MountingHole:MountingHole_4.3mm_M4_Pad, F.Cu at (292.0, 5.00)
- added REF**: MountingHole_4.3mm_M4_Pad, MountingHole:MountingHole_4.3mm_M4_Pad, F.Cu at (4.00, 5.00)
- added REF**: MountingHole_4.3mm_M4_Pad, MountingHole:MountingHole_4.3mm_M4_Pad, F.Cu at (5.00, 204.0)
- added REF**: MountingHole_4.3mm_M4_Pad, MountingHole:MountingHole_4.3mm_M4_Pad, F.Cu at (292.0, 205.0)
- added RV1: R_Potentiometer, Potentiometer_THT:Potentiometer_ACP_CA6-H2,5_Horizontal, F.Cu at (255.7, 52.5)
- C4: value 470μF -> C_Polarized
- C6: value 10000μF -> C_Polarized
- J10: value SIM 900D Connector -> Conn_01x03_Female
- J11: value Lamp Connector -> Conn_WallSocket
- J12: value Padding Wheel Connector -> Conn_WallSocket
- J8: value LCD Connector -> Conn_01x16_Male; footprint Connector_PinSocket_2.54mm:PinSocket_1x14_P2.54mm_Vertical -> Connector_PinHeader_2.54mm:PinHeader_1x16_P2.54mm_Vertical
- J9: value 12V AC SUPPLY -> Conn_01x02_Female
- L1: value 27uH -> INDUCTOR
- M2: value Servo Motor Connector -> Motor_Servo
- R5, R6, R7, R8: value 10K -> R
- RL1: value Lamp Control Relay -> FINDER-36.11
- RL2: value Padding Wheel Control Relay -> FINDER-36.11
- U2: value LM7809 -> LM7809_TO220
- U3: value LM7812 -> LM7812_TO220
- U4: value ATmega32 -> ATmega32A-P
- U5: value L293D Motor Controller -> L293D
- U7: value DS3232M RTC -> DS3232M
- U8: value PCF8574 I2C to 8bit -> PCF8574
- Ultrasonic1: value Ultrasonic Connector -> Conn_01x04_Female
Connections:
- J8 pad 1: unconnected-(J8-Pad1) -> Net-(BZ1-Pad2)
- J8 pad 10: unconnected-(J8-Pad10) -> Net-(BZ1-Pad2)
- J8 pad 3: unconnected-(J8-Pad3) -> Net-(J8-Pad3)
- J8 pad 7: unconnected-(J8-Pad7) -> Net-(BZ1-Pad2)
- J8 pad 8: unconnected-(J8-Pad8) -> Net-(BZ1-Pad2)
- J8 pad 9: unconnected-(J8-Pad9) -> Net-(BZ1-Pad2)
Routing:
- net Net-(J8-Pad3): track 0.00 -> 72.4 mm, vias 0 -> 1
- net Net-(BZ1-Pad2): track 1336.3 -> 1362.7 mm
- net Net-(C3-Pad1): track 898.7 -> 908.9 mm
- net Net-(J7-Pad1): track 159.9 -> 168.1 mm
- net Net-(J7-Pad2): track 153.4 -> 160.6 mm
- net Net-(J7-Pad4): track 138.1 -> 145.1 mm
- net Net-(J7-Pad3): track 145.9 -> 152.8 mm
- net Net-(RL1-PadA1): track 156.0 -> 162.0 mm
- net Net-(J7-Pad8): track 138.3 -> 132.9 mm
- net Net-(J7-Pad7): track 136.0 -> 131.9 mm
- net Net-(U4-Pad17): track 213.4 -> 210.5 mm
- net Net-(J7-Pad6): track 133.8 -> 131.6 mm
- net Net-(HX1-Pad11): track 134.7 -> 135.9 mm
- net Net-(U4-Pad16): track 218.6 -> 217.3 mm
- net Net-(RL2-PadA1): track 219.2 -> 218.1 mm
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- added copper zone on B.Cu, net (none)
- added copper zone on F.Cu, net (none)
- removed copper zone on F.Cu, net Net-(C3-Pad1)
Other:
- board text added: "SIM 900D 190x160"
- board text removed: "SIM 900D"

Commit message: add
Routing:
- net Net-(BZ1-Pad2): track 1362.7 -> 1463.0 mm
- net Net-(HX1-Pad10): track 0.00 -> 26.3 mm
- net Net-(R5-Pad1): track 227.6 -> 215.2 mm
- net Net-(R6-Pad1): track 224.6 -> 214.4 mm
- net Net-(C3-Pad1): track 908.9 -> 904.1 mm
- net Net-(J7-Pad5): track 131.1 -> 129.9 mm
- added copper zone on B.Cu, net Net-(BZ1-Pad2)
- added copper zone on F.Cu, net Net-(BZ1-Pad2)
- removed copper zone on B.Cu, net (none)
- removed copper zone on F.Cu, net (none)
- removed copper zone on B.Cu, net Net-(C3-Pad1)
Other:
- board text added: "S0"
- board text removed: "Signal"
