File: GSM_LCD_RTC/GSM_LCD_RTC.kicad_sch (KiCad schematic)
At the start: 10 parts, among them J1 Screw_Terminal_01x02, J2 Conn_01x14_Female, U1 ATmega32A-P, U2 PCF8574, U3 DS3232M, U5 SIM900

Commit message: add
Parts:
- removed U5: SIM900, RF_GSM:SIMCom_SIM900, symbol RF_GSM:SIM900
- added J3: Conn_01x03_Female, Connector_PinSocket_2.54mm:PinSocket_1x03_P2.54mm_Vertical, symbol Connector:Conn_01x03_Female
- J1: footprint Connector_PinSocket_2.54mm:PinSocket_1x02_P2.54mm_Vertical -> Connector_PinSocket_2.54mm:PinSocket_1x03_P2.54mm_Vertical
Connections:
- net at J1.2 (Pin_2), U1.11 (GND), U1.31 (GND)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: now also J3.3 (Pin_3)
- net at U1.14 (PD0): now also J3.1 (Pin_1)
- net at U1.15 (PD1): now also J3.2 (Pin_2)
Changed lines of the file:
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@@
   (junction (at 111.76 163.83) (diameter 0) (color 0 0 0 0)
   )
+  (junction (at 171.45 128.27) (diameter 0) (color 0 0 0 0)
+  )
   (junction (at 138.43 82.55) (diameter 0) (color 0 0 0 0)
   )
@@
   (junction (at 152.4 16.51) (diameter 0) (color 0 0 0 0)
   )
-  (junction (at 171.45 163.83) (diameter 0) (color 0 0 0 0)
-  )
   (junction (at 119.38 38.1) (diameter 0) (color 0 0 0 0)
   )
   (junction (at 143.51 85.09) (diameter 0) (color 0 0 0 0)
   )
-  (junction (at 236.22 160.02) (diameter 0) (color 0 0 0 0)
-  )
   (junction (at 138.43 106.68) (diameter 0) (color 0 0 0 0)
   )
@@
     (stroke (width 0) (type default) (color 0 0 0 0))
   )
-  (wire (pts (xy 236.22 160.02) (xy 236.22 163.83))
-    (stroke (width 0) (type default) (color 0 0 0 0))
-  )
   (wire (pts (xy 135.89 39.37) (xy 135.89 41.91))
     (stroke (width 0) (type default) (color 0 0 0 0))
@@
     (stroke (width 0) (type default) (color 0 0 0 0))
   )
-  (wire (pts (xy 198.12 101.6) (xy 218.44 101.6))
-    (stroke (width 0) (type default) (color 0 0 0 0))
-  )
-  (wire (pts (xy 236.22 163.83) (xy 171.45 163.83))
+  (wire (pts (xy 198.12 101.6) (xy 234.95 101.6))
     (stroke (width 0) (type default) (color 0 0 0 0))
   )
@@
     (stroke (width 0) (type default) (color 0 0 0 0))
   )
-  (wire (pts (xy 236.22 157.48) (xy 236.22 160.02))
-    (stroke (width 0) (type default) (color 0 0 0 0))
-  )
   (wire (pts (xy 179.07 49.53) (xy 218.44 49.53))
     (stroke (width 0) (type default) (color 0 0 0 0))
@@
     (stroke (width 0) (type default) (color 0 0 0 0))
   )
-  (wire (pts (xy 171.45 97.79) (xy 171.45 163.83))
+  (wire (pts (xy 205.74 106.68) (xy 205.74 128.27))
+    (stroke (width 0) (type default) (color 0 0 0 0))
+  )
+  (wire (pts (xy 171.45 97.79) (xy 171.45 128.27))
     (stroke (width 0) (type default) (color 0 0 0 0))
   )
@@
     (stroke (width 0) (type default) (color 0 0 0 0))
   )
+  (wire (pts (xy 205.74 128.27) (xy 171.45 128.27))
+    (stroke (width 0) (type default) (color 0 0 0 0))
+  )
   (wire (pts (xy 139.7 36.83) (xy 135.89 36.83))
     (stroke (width 0) (type default) (color 0 0 0 0))
@@
     (stroke (width 0) (type default) (color 0 0 0 0))
   )
+  (wire (pts (xy 171.45 128.27) (xy 171.45 163.83))
+    (stroke (width 0) (type default) (color 0 0 0 0))
+  )
   (wire (pts (xy 198.12 123.19) (xy 77.47 123.19))
     (stroke (width 0) (type default) (color 0 0 0 0))
@@
     (stroke (width 0) (type default) (color 0 0 0 0))
   )
+  (wire (pts (xy 234.95 106.68) (xy 205.74 106.68))
+    (stroke (width 0) (type default) (color 0 0 0 0))
+  )
   (wire (pts (xy 187.96 29.21) (xy 187.96 26.67))
     (stroke (width 0) (type default) (color 0 0 0 0))
@@
     (stroke (width 0) (type default) (color 0 0 0 0))
   )
-  (wire (pts (xy 201.93 104.14) (xy 218.44 104.14))
-    (stroke (width 0) (type default) (color 0 0 0 0))
+  (wire (pts (xy 201.93 104.14) (xy 234.95 104.14))
+    (stroke (width 0) (type default) (color 0 0 0 0))
+  )
+  (symbol (lib_id "Connector:Conn_01x03_Female") (at 240.03 104.14 0) (unit 1)
+    (in_bom yes) (on_board yes) (fields_autoplaced)
+    (property "Reference" "J3" (id 0) (at 241.3 102.8699 0)
+      (effects (font (size 1.27 1.27)) (justify left))
+    )
+    (property "Value" "Conn_01x03_Female" (id 1) (at 241.3 105.4099 0)
+      (effects (font (size 1.27 1.27)) (justify left))
+    )
+    (property "Footprint" "Connector_PinSocket_2.54mm:PinSocket_1x03_P2.54mm_Vertical" (id 2) (at 240.03 104.14 0)
+      (effects (font (size 1.27 1.27)) hide)
+    )
+    (property "Datasheet" "~" (id 3) (at 240.03 104.14 0)
+      (effects (font (size 1.27 1.27)) hide)
+    )
+    (pin "1")
+    (pin "2")
+    (pin "3")
   )
   (symbol (lib_id "Device:R") (at 143.51 93.98 0) (unit 1)
@@
       (effects (font (size 1.27 1.27)) (justify left))
     )
-    (property "Footprint" "Connector_PinSocket_2.54mm:PinSocket_1x02_P2.54mm_Vertical" (id 2) (at 114.3 181.61 0)
+    (property "Footprint" "Connector_PinSocket_2.54mm:PinSocket_1x03_P2.54mm_Vertical" (id 2) (at 114.3 181.61 0)
       (effects (font (size 1.27 1.27)) hide)
     )
@@
     (pin "2")
   )
-  (symbol (lib_id "RF_GSM:SIM900") (at 236.22 119.38 0) (unit 1)
-    (in_bom yes) (on_board yes) (fields_autoplaced)
-    (property "Reference" "U5" (id 0) (at 238.2394 160.02 0)
-      (effects (font (size 1.27 1.27)) (justify left))
-    )
-    (property "Value" "SIM900" (id 1) (at 238.2394 162.56 0)
-      (effects (font (size 1.27 1.27)) (justify left))
-    )
-    (property "Footprint" "RF_GSM:SIMCom_SIM900" (id 2) (at 248.92 158.75 0)
-      (effects (font (size 1.27 1.27)) hide)
-    )
-    (property "Datasheet" "http://simcom.ee/documents/SIM900/SIM900_Hardware%20Design_V2.05.pdf" (id 3) (at 185.42 86.36 0)
+  (symbol (lib_id "Interface_Expansion:PCF8574") (at 152.4 39.37 0) (unit 1)
+    (in_bom yes) (on_board yes) (fields_autoplaced)
+    (property "Reference" "U2" (id 0) (at 154.4194 19.05 0)
+      (effects (font (size 1.27 1.27)) (justify left))
+    )
+    (property "Value" "PCF8574" (id 1) (at 154.4194 21.59 0)
+      (effects (font (size 1.27 1.27)) (justify left))
+    )
+    (property "Footprint" "Module:Pololu_Breakout-16_15.2x20.3mm" (id 2) (at 152.4 39.37 0)
+      (effects (font (size 1.27 1.27)) hide)
+    )
+    (property "Datasheet" "http://www.nxp.com/documents/data_sheet/PCF8574_PCF8574A.pdf" (id 3) (at 152.4 39.37 0)
       (effects (font (size 1.27 1.27)) hide)
     )
@@
     (pin "15")
     (pin "16")
-    (pin "17")
-    (pin "18")
-    (pin "19")
-    (pin "2")
-    (pin "20")
-    (pin "21")
-    (pin "22")
-    (pin "23")
-    (pin "24")
-    (pin "25")
-    (pin "26")
-    (pin "27")
-    (pin "28")
-    (pin "29")
-    (pin "3")
-    (pin "30")
-    (pin "31")
-    (pin "32")
-    (pin "33")
-    (pin "34")
-    (pin "35")
-    (pin "36")
-    (pin "37")
-    (pin "38")
-    (pin "39")
-    (pin "4")
-    (pin "40")
-    (pin "41")
-    (pin "42")
-    (pin "43")
-    (pin "44")
-    (pin "45")
-    (pin "46")
-    (pin "47")
-    (pin "48")
-    (pin "49")
-    (pin "5")
-    (pin "50")
-    (pin "51")
-    (pin "52")
-    (pin "53")
-    (pin "54")
-    (pin "55")
-    (pin "56")
-    (pin "57")
-    (pin "58")
-    (pin "59")
-    (pin "6")
-    (pin "60")
-    (pin "61")
-    (pin "62")
-    (pin "63")
-    (pin "64")
-    (pin "65")
-    (pin "66")
-    (pin "67")
-    (pin "68")
-    (pin "7")
-    (pin "8")
-    (pin "9")
-  )
-  (symbol (lib_id "Interface_Expansion:PCF8574") (at 152.4 39.37 0) (unit 1)
-    (in_bom yes) (on_board yes) (fields_autoplaced)
-    (property "Reference" "U2" (id 0) (at 154.4194 19.05 0)
-      (effects (font (size 1.27 1.27)) (justify left))
-    )
-    (property "Value" "PCF8574" (id 1) (at 154.4194 21.59 0)
-      (effects (font (size 1.27 1.27)) (justify left))
-    )
-    (property "Footprint" "Module:Pololu_Breakout-16_15.2x20.3mm" (id 2) (at 152.4 39.37 0)
-      (effects (font (size 1.27 1.27)) hide)
-    )
-    (property "Datasheet" "http://www.nxp.com/documents/data_sheet/PCF8574_PCF8574A.pdf" (id 3) (at 152.4 39.37 0)
-      (effects (font (size 1.27 1.27)) hide)
-    )
-    (pin "1")
-    (pin "10")
-    (pin "11")
-    (pin "12")
-    (pin "13")
-    (pin "14")
-    (pin "15")
-    (pin "16")
     (pin "2")
     (pin "3")
@@
   (symbol_instances
     (path "/e4aa07eb-0025-4c9a-b1bf-7c0fd782aa3e"
-      (reference "J1") (unit 1) (value "Screw_Terminal_01x02") (footprint "Connector_PinSocket_2.54mm:PinSocket_1x02_P2.54mm_Vertical")
+      (reference "J1") (unit 1) (value "Screw_Terminal_01x02") (footprint "Connector_PinSocket_2.54mm:PinSocket_1x03_P2.54mm_Vertical")
     )
     (path "/c463bf48-a5c3-44e4-a3a1-2dd23614d398"
       (reference "J2") (unit 1) (value "Conn_01x14_Female") (footprint "Connector_PinSocket_2.54mm:PinSocket_1x14_P2.54mm_Vertical")
     )
+    (path "/4eae46a2-a55c-4f91-9111-48ccc1e331be"
+      (reference "J3") (unit 1) (value "Conn_01x03_Female") (footprint "Connector_PinSocket_2.54mm:PinSocket_1x03_P2.54mm_Vertical")
+    )
     (path "/db648446-8adf-4fce-92e0-5e6f32f62abc"
       (reference "R1") (unit 1) (value "R") (footprint "Resistor_THT:R_Axial_DIN0411_L9.9mm_D3.6mm_P20.32mm_Horizontal")
@@
       (reference "U3") (unit 1) (value "DS3232M") (footprint "Package_SO:SOIC-8_3.9x4.9mm_P1.27mm")
     )
-    (path "/e5d2dd88-0dc9-48f4-ab55-fd452ef5df07"
-      (reference "U5") (unit 1) (value "SIM900") (footprint "RF_GSM:SIMCom_SIM900")
-    )
-  )
+  )

Commit message: add
Parts:
- J1: footprint Connector_PinSocket_2.54mm:PinSocket_1x03_P2.54mm_Vertical -> Connector_PinSocket_2.54mm:PinSocket_1x02_P2.54mm_Vertical
Changed lines of the file:
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@@
       (effects (font (size 1.27 1.27)) (justify left))
     )
-    (property "Footprint" "Connector_PinSocket_2.54mm:PinSocket_1x03_P2.54mm_Vertical" (id 2) (at 114.3 181.61 0)
+    (property "Footprint" "Connector_PinSocket_2.54mm:PinSocket_1x02_P2.54mm_Vertical" (id 2) (at 114.3 181.61 0)
       (effects (font (size 1.27 1.27)) hide)
     )
@@
   (symbol_instances
     (path "/e4aa07eb-0025-4c9a-b1bf-7c0fd782aa3e"
-      (reference "J1") (unit 1) (value "Screw_Terminal_01x02") (footprint "Connector_PinSocket_2.54mm:PinSocket_1x03_P2.54mm_Vertical")
+      (reference "J1") (unit 1) (value "Screw_Terminal_01x02") (footprint "Connector_PinSocket_2.54mm:PinSocket_1x02_P2.54mm_Vertical")
     )
     (path "/c463bf48-a5c3-44e4-a3a1-2dd23614d398"

Commit message: add
Parts:
- removed J2: Conn_01x14_Female, Connector_PinSocket_2.54mm:PinSocket_1x14_P2.54mm_Vertical, symbol Connector:Conn_01x14_Female
- added J2: LCD Connector, Connector_PinHeader_2.54mm:PinHeader_1x16_P2.54mm_Vertical, symbol Connector:Conn_01x16_Female
- added RV1: R_Potentiometer, symbol Device:R_Potentiometer
- J1: value Screw_Terminal_01x02 -> Power IN; footprint Connector_PinSocket_2.54mm:PinSocket_1x02_P2.54mm_Vertical -> Connector_Phoenix_MSTB:PhoenixContact_MSTBA_2,5_2-G_1x02_P5.00mm_Horizontal
- J3: value Conn_01x03_Female -> GSM Connecetor
Connections:
- net at J1.2 (Pin_2), J3.3 (Pin_3), U1.11 (GND)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: now also J2.1 (Pin_1), J2.10 (Pin_10), J2.16 (Pin_16), J2.7 (Pin_7), J2.8 (Pin_8), J2.9 (Pin_9), RV1.3
- net at J1.1 (Pin_1), R1.2, R2.2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: now also J2.15 (Pin_15), J2.2 (Pin_2), RV1.1
- net at U2.9 (P4): now also J2.11 (Pin_11)
- net at U2.10 (P5): now also J2.12 (Pin_12)
- net at U2.11 (P6): now also J2.13 (Pin_13)
- net at U2.12 (P7): now also J2.14 (Pin_14)
- net at U2.4 (P0): now also J2.4 (Pin_4)
- net at U2.5 (P1): now also J2.5 (Pin_5)
- net at U2.6 (P2): now also J2.6 (Pin_6)
- new net: J2.3 (Pin_3), RV1.2

Commit message: lcd
Parts:
- RV1: value R_Potentiometer -> 10K Potentiometer; footprint (none) -> Potentiometer_THT:Potentiometer_ACP_CA6-H2,5_Horizontal
Changed lines of the file:
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@@
       (effects (font (size 1.27 1.27)) (justify right))
     )
-    (property "Value" "R_Potentiometer" (id 1) (at 205.74 36.8299 0)
+    (property "Value" "10K Potentiometer" (id 1) (at 205.74 36.8299 0)
       (effects (font (size 1.27 1.27)) (justify right))
     )
-    (property "Footprint" "" (id 2) (at 208.28 35.56 0)
+    (property "Footprint" "Potentiometer_THT:Potentiometer_ACP_CA6-H2,5_Horizontal" (id 2) (at 208.28 35.56 0)
       (effects (font (size 1.27 1.27)) hide)
     )
@@
     )
     (path "/b482f951-6b79-4727-885d-127f4f445c7d"
-      (reference "RV1") (unit 1) (value "R_Potentiometer") (footprint "Potentiometer_THT:Potentiometer_ACP_CA6-H2,5_Horizontal")
+      (reference "RV1") (unit 1) (value "10K Potentiometer") (footprint "Potentiometer_THT:Potentiometer_ACP_CA6-H2,5_Horizontal")
     )
     (path "/7dac8009-a015-44c1-ab8b-d0d637a9bdd9"
