File: GSM_LCD_RTC/GSM_LCD_RTC.kicad_pcb (KiCad board)
At the start: 4 copper layers, 15 parts, among them J1 Screw_Terminal_01x02, J2 Conn_01x14_Female, U1 ATmega32A-P, U2 PCF8574, U3 DS3232M, U5 SIM900

Commit message: add
Parts:
- removed U5: SIM900, RF_GSM:SIMCom_SIM900
- added J3: Conn_01x03_Female, Connector_PinSocket_2.54mm:PinSocket_1x03_P2.54mm_Vertical, F.Cu at (154.8, 137.5)
- J1: footprint Connector_PinSocket_2.54mm:PinSocket_1x02_P2.54mm_Vertical -> Connector_PinSocket_2.54mm:PinSocket_1x03_P2.54mm_Vertical
Routing:
- net Net-(J1-Pad2): track 502.3 -> 474.0 mm, vias 2 -> 1
- net Net-(U1-Pad14): track 219.8 -> 212.7 mm, vias 1 -> 0
- net Net-(U1-Pad15): track 239.3 -> 233.3 mm, vias 1 -> 0
Other:
- board text added: "GSM Module"

Commit message: add
Parts:
- removed REF** (x5): MountingHole_5.3mm_M5, MountingHole:MountingHole_5.3mm_M5
- J1: footprint Connector_PinSocket_2.54mm:PinSocket_1x03_P2.54mm_Vertical -> Connector_PinSocket_2.54mm:PinSocket_1x02_P2.54mm_Vertical
- moved J1 97.1 mm to (51.0, 187.3)
- moved R4 89.0 mm to (111.4, 137.0), turned to -90 degrees
- moved R3 77.3 mm to (130.0, 136.6), turned to -90 degrees
- moved R1 71.2 mm to (129.0, 92.3), turned to -90 degrees
- moved R2 45.1 mm to (113.6, 92.1), turned to -90 degrees
- moved U2 44.8 mm to (148.3, 80.5)
- moved U1 42.2 mm to (72.1, 67.8)
- moved U3 36.7 mm to (150.0, 118.0)
- moved J2 31.6 mm to (205.4, 72.8), turned to 0 degrees
- moved J3 27.4 mm to (176.6, 120.9), turned to 0 degrees
Routing:
- net Net-(J1-Pad1): track 1346.6 -> 587.8 mm, vias 0 -> 3
- net Net-(J2-Pad5): track 211.2 -> 127.1 mm
- net Net-(J2-Pad6): track 197.5 -> 113.9 mm
- net Net-(J2-Pad4): track 222.8 -> 139.2 mm
- net Net-(R1-Pad1): track 338.7 -> 269.0 mm
- net Net-(J2-Pad11): track 110.7 -> 44.5 mm
- net Net-(J2-Pad12): track 108.3 -> 48.2 mm, vias 0 -> 2
- net Net-(J2-Pad13): track 103.8 -> 50.6 mm, vias 0 -> 2
- net Net-(J2-Pad14): track 98.7 -> 54.6 mm, vias 0 -> 2
- net Net-(R2-Pad1): track 360.7 -> 320.5 mm, vias 1 -> 2
- net Net-(J3-Pad1): track 212.7 -> 237.8 mm, vias 0 -> 1
- net Net-(J1-Pad2): track 474.0 -> 486.5 mm
- net Net-(J3-Pad2): track 233.3 -> 223.0 mm, vias 0 -> 1
- added copper zone on B.Cu, net (none)
- added copper zone on F.Cu, net (none)
Other:
- copper layers 4 -> 2
- board text removed: "16x2 LCD DISPLAY"
- board text removed: "GND"
- board text removed: "GSM Module"
- board text removed: "VCC +5V"

Commit message: add
Parts:
- added REF**: MountingHole_4.3mm_M4, MountingHole:MountingHole_4.3mm_M4, F.Cu at (237.0, 167.0)
- added REF**: MountingHole_4.3mm_M4, MountingHole:MountingHole_4.3mm_M4, F.Cu at (40.0, 26.0)
- added REF**: MountingHole_4.3mm_M4, MountingHole:MountingHole_4.3mm_M4, F.Cu at (236.0, 26.0)
- added REF**: MountingHole_4.3mm_M4, MountingHole:MountingHole_4.3mm_M4, F.Cu at (41.0, 167.0)
- R1, R2, R3, R4: value R -> 10K
- U1: value ATmega32A-P -> ATmega32
- moved J1 34.4 mm to (53.6, 153.0)
- moved R1 34.4 mm to (131.6, 58.0)
- moved U1 34.4 mm to (74.7, 33.5)
- moved U2 34.4 mm to (150.9, 46.2)
- moved J2 34.4 mm to (208.0, 38.5)
- moved J3 34.4 mm to (179.2, 86.6)
- moved R2 34.4 mm to (116.2, 57.8)
- moved R3 34.4 mm to (132.6, 102.3)
- moved R4 34.4 mm to (114.0, 102.7)
- moved U3 34.4 mm to (152.6, 83.7)
Routing:
- net Net-(R1-Pad1): track 269.0 -> 295.1 mm
Other:
- board text added: "+5V"
- board text added: "D4"
- board text added: "D5"
- board text added: "D6"
- board text added: "D7"
- board text added: "E"
- board text added: "GND"
- board text added: "RS"
- board text added: "RW"
- board text added: "RXD"
- board text added: "TXD"
- board text added: "VDD"

Commit message: add
Parts:
- added RV1: R_Potentiometer, Potentiometer_THT:Potentiometer_ACP_CA6-H2,5_Horizontal, F.Cu at (234.0, 57.0)
- J1: value Screw_Terminal_01x02 -> Power IN; footprint Connector_PinSocket_2.54mm:PinSocket_1x02_P2.54mm_Vertical -> Connector_Phoenix_MSTB:PhoenixContact_MSTBA_2,5_2-G_1x02_P5.00mm_Horizontal
- J2: value Conn_01x14_Female -> LCD Connector; footprint Connector_PinSocket_2.54mm:PinSocket_1x14_P2.54mm_Vertical -> Connector_PinHeader_2.54mm:PinHeader_1x16_P2.54mm_Vertical
- J3: value Conn_01x03_Female -> GSM Connecetor
- R1, R2, R3, R4: value 10K -> R
- U1: value ATmega32 -> ATmega32A-P
- moved REF** 14.0 mm to (250.0, 26.0)
- moved REF** 13.0 mm to (250.0, 167.0)
Connections:
- J2 pad 1: unconnected-(J2-Pad1) -> Net-(J1-Pad2)
- J2 pad 10: unconnected-(J2-Pad10) -> Net-(J1-Pad2)
- J2 pad 3: unconnected-(J2-Pad3) -> Net-(RV1-Pad2)
- J2 pad 7: unconnected-(J2-Pad7) -> Net-(J1-Pad2)
- J2 pad 8: unconnected-(J2-Pad8) -> Net-(J1-Pad2)
- J2 pad 9: unconnected-(J2-Pad9) -> Net-(J1-Pad2)
Routing:
- net Net-(J1-Pad1): track 587.8 -> 793.6 mm
- net Net-(J1-Pad2): track 486.5 -> 691.4 mm, vias 1 -> 2
- net Net-(U2-Pad5): track 127.1 -> 0.00 mm
- net Net-(U2-Pad6): track 113.9 -> 0.00 mm
- net Net-(RV1-Pad2): track 0.00 -> 29.2 mm

Commit message: add
Parts:
- moved J1 4.00 mm to (53.5, 157.0), turned to 0 degrees
Routing:
- net Net-(J1-Pad2): track 691.4 -> 697.9 mm
- net Net-(J1-Pad1): track 793.6 -> 797.3 mm

Commit message: add
Parts:
- moved J1 16.0 mm to (69.0, 153.0)
Routing:
- net Net-(J1-Pad1): track 797.3 -> 811.7 mm
- net Net-(J1-Pad2): track 697.9 -> 707.3 mm
Changed lines of the file:
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@@
   )
   (footprint "Connector_Phoenix_MSTB:PhoenixContact_MSTBA_2,5_2-G_1x02_P5.00mm_Horizontal" (layer "F.Cu")
-    (at 53.5 157)
+    (at 69 153)
     (descr "Generic Phoenix Contact connector footprint for: MSTBA_2,5/2-G; number of pins: 02; pin pitch: 5.00mm; Angled || order number: 1757475 12A || order number: 1923759 16A (HC)")
     (tags "phoenix_contact connector MSTBA_01x02_G_5.00mm")
@@
     (effects (font (size 1 1) (thickness 0.15)))
   )
-  (gr_text "GND" (at 61 165) (layer "F.SilkS")
+  (gr_text "GND" (at 75 166) (layer "F.SilkS")
     (effects (font (size 2 2) (thickness 0.4)))
   )
@@
     (effects (font (size 1 1) (thickness 0.15)))
   )
-  (gr_text "+5V" (at 54 165) (layer "F.SilkS")
+  (gr_text "+5V" (at 68 166) (layer "F.SilkS")
     (effects (font (size 2 2) (thickness 0.4)))
   )
@@
   (segment (start 131.36 78.12) (end 131.6 78.36) (width 1) (layer "B.Cu") (net 1))
   (segment (start 146.46 46.21) (end 150.86 46.21) (width 1) (layer "B.Cu") (net 1))
+  (segment (start 47.5 151) (end 49.5 153) (width 1) (layer "B.Cu") (net 1))
   (segment (start 146.46 51.29) (end 150.86 51.29) (width 1) (layer "B.Cu") (net 1))
   (segment (start 142.1 116.2) (end 142.1 86.6) (width 1) (layer "B.Cu") (net 1))
@@
   (segment (start 148.5 59.5) (end 148.5 70.2) (width 0.8) (layer "B.Cu") (net 1))
   (segment (start 144.8 40.9) (end 149.2 40.9) (width 1) (layer "B.Cu") (net 1))
-  (segment (start 53.6 60.5) (end 53.6 148.4) (width 1) (layer "B.Cu") (net 1))
   (segment (start 141.5 53) (end 143.11 51.39) (width 1) (layer "B.Cu") (net 1))
-  (segment (start 47.5 151) (end 50 153.5) (width 1) (layer "B.Cu") (net 1))
-  (segment (start 53.6 148.4) (end 50 152) (width 1) (layer "B.Cu") (net 1))
-  (segment (start 50 153.5) (end 53.5 157) (width 1) (layer "B.Cu") (net 1))
+  (segment (start 74.675 56.335) (end 57.765 56.335) (width 1) (layer "B.Cu") (net 1))
+  (segment (start 58 153) (end 69 153) (width 1) (layer "B.Cu") (net 1))
   (segment (start 132.2 123.02) (end 132.6 122.62) (width 1) (layer "B.Cu") (net 1))
   (segment (start 149.2 40.9) (end 149.3 40.8) (width 1) (layer "B.Cu") (net 1))
-  (segment (start 74.675 56.335) (end 57.765 56.335) (width 1) (layer "B.Cu") (net 1))
   (segment (start 143.11 51.39) (end 146.36 51.39) (width 1) (layer "B.Cu") (net 1))
-  (segment (start 57.765 56.335) (end 53.6 60.5) (width 1) (layer "B.Cu") (net 1))
-  (segment (start 50 153) (end 50 152) (width 1) (layer "B.Cu") (net 1))
   (segment (start 214.8 74.5) (end 217.1 72.2) (width 0.8) (layer "B.Cu") (net 1))
   (segment (start 162.2 40.8) (end 162.3 40.7) (width 1) (layer "B.Cu") (net 1))
-  (segment (start 50.7 131.8) (end 50.2 132.3) (width 1) (layer "B.Cu") (net 1))
+  (segment (start 53.6 148.6) (end 58 153) (width 1) (layer "B.Cu") (net 1))
   (segment (start 162.3 40.7) (end 207.66 40.7) (width 1) (layer "B.Cu") (net 1))
   (segment (start 217.1 72.2) (end 217.1 53) (width 0.8) (layer "B.Cu") (net 1))
@@
   (segment (start 146.36 46.31) (end 146.46 46.21) (width 1) (layer "B.Cu") (net 1))
   (segment (start 116.2 78.12) (end 131.36 78.12) (width 1) (layer "B.Cu") (net 1))
+  (segment (start 57.765 56.335) (end 53.6 60.5) (width 1) (layer "B.Cu") (net 1))
+  (segment (start 47.5 92.5) (end 47.5 151) (width 1) (layer "B.Cu") (net 1))
   (segment (start 135.6 122.7) (end 142.1 116.2) (width 1) (layer "B.Cu") (net 1))
   (segment (start 141.5 50.4) (end 143.05 48.85) (width 1) (layer "B.Cu") (net 1))
+  (segment (start 53.6 60.5) (end 53.6 148.6) (width 1) (layer "B.Cu") (net 1))
   (segment (start 215.3 51.2) (end 208 51.2) (width 0.8) (layer "B.Cu") (net 1))
   (segment (start 146.36 51.39) (end 146.46 51.29) (width 1) (layer "B.Cu") (net 1))
   (segment (start 149.3 40.8) (end 162.2 40.8) (width 1) (layer "B.Cu") (net 1))
-  (segment (start 50.2 132.3) (end 50.2 152.8) (width 1) (layer "B.Cu") (net 1))
   (segment (start 141.5 44.2) (end 144.8 40.9) (width 1) (layer "B.Cu") (net 1))
   (segment (start 141.5 76.4) (end 141.5 53) (width 1) (layer "B.Cu") (net 1))
+  (segment (start 50.2 132.3) (end 50.2 148) (width 1) (layer "B.Cu") (net 1))
   (segment (start 146.46 48.75) (end 150.86 48.75) (width 1) (layer "B.Cu") (net 1))
-  (segment (start 47.5 92.5) (end 47.5 151) (width 1) (layer "B.Cu") (net 1))
-  (segment (start 50.2 152.8) (end 50 153) (width 1) (layer "B.Cu") (net 1))
-  (segment (start 49.8 90.2) (end 47.5 92.5) (width 1) (layer "B.Cu") (net 1))
+  (segment (start 50.7 131.8) (end 50.2 132.3) (width 1) (layer "B.Cu") (net 1))
   (segment (start 141.5 47.4) (end 141.5 44.2) (width 1) (layer "B.Cu") (net 1))
   (segment (start 217.1 53) (end 215.3 51.2) (width 0.8) (layer "B.Cu") (net 1))
   (segment (start 150.86 58.91) (end 149.51 58.91) (width 0.8) (layer "B.Cu") (net 1))
-  (segment (start 50 152) (end 50 153.5) (width 1) (layer "B.Cu") (net 1))
+  (segment (start 50.2 148) (end 55 152.8) (width 1) (layer "B.Cu") (net 1))
+  (segment (start 49.5 153) (end 58 153) (width 1) (layer "B.Cu") (net 1))
   (segment (start 143.05 48.85) (end 146.36 48.85) (width 1) (layer "B.Cu") (net 1))
   (segment (start 162.2 40.8) (end 163.56 42.16) (width 1) (layer "B.Cu") (net 1))
@@
   (segment (start 148.5 70.2) (end 152.8 74.5) (width 0.8) (layer "B.Cu") (net 1))
   (segment (start 141.5 53) (end 141.5 50.4) (width 1) (layer "B.Cu") (net 1))
+  (segment (start 49.8 90.2) (end 47.5 92.5) (width 1) (layer "B.Cu") (net 1))
   (segment (start 141.5 50.4) (end 141.5 47.4) (width 1) (layer "B.Cu") (net 1))
   (segment (start 208 58.82) (end 208 61.36) (width 0.5) (layer "F.Cu") (net 2))
@@
   (segment (start 219.1 51.7) (end 216.06 48.66) (width 0.8) (layer "B.Cu") (net 2))
   (segment (start 151.9 76.3) (end 215.6 76.3) (width 0.8) (layer "B.Cu") (net 2))
+  (segment (start 58.5 149.5) (end 70.5 149.5) (width 1) (layer "B.Cu") (net 2))
   (segment (start 208 88) (end 208 82) (width 1) (layer "B.Cu") (net 2))
   (segment (start 148.73 56.37) (end 146.8 58.3) (width 0.8) (layer "B.Cu") (net 2))
@@
   (segment (start 59.425 58.875) (end 56.14 62.16) (width 1) (layer "B.Cu") (net 2))
   (segment (start 171.9 131.7) (end 164.1 139.5) (width 1) (layer "B.Cu") (net 2))
-  (segment (start 58.5 149.5) (end 58.5 157) (width 1) (layer "B.Cu") (net 2))
   (segment (start 146.8 71.2) (end 151.9 76.3) (width 0.8) (layer "B.Cu") (net 2))
+  (segment (start 70.5 149.5) (end 74 153) (width 1) (layer "B.Cu") (net 2))
   (segment (start 168.499511 90.299511) (end 168.499511 130.600489) (width 1) (layer "B.Cu") (net 2))
   (segment (start 168.499511 130.600489) (end 162.1 137) (width 1) (layer "B.Cu") (net 2))

Commit message: lcd
Parts:
- RV1: value R_Potentiometer -> 10K Potentiometer
Routing:
- net Net-(J1-Pad2): track 707.3 -> 580.2 mm
- net Net-(J1-Pad1): track 811.7 -> 697.8 mm
- net Net-(J2-Pad5): track 0.00 -> 106.6 mm, vias 0 -> 2
- net Net-(J2-Pad6): track 0.00 -> 97.3 mm, vias 0 -> 2

Commit message: add
Routing:
- net Net-(J1-Pad2): track 580.2 -> 607.0 mm
- net Net-(J2-Pad4): track 139.2 -> 140.1 mm
Changed lines of the file:
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@@
   (segment (start 74.675 58.875) (end 59.425 58.875) (width 1) (layer "B.Cu") (net 2))
   (segment (start 162.1 137) (end 62.2 137) (width 1) (layer "B.Cu") (net 2))
+  (segment (start 212.4 76.6) (end 215 74) (width 1) (layer "B.Cu") (net 2))
   (segment (start 58.5 149.5) (end 70.5 149.5) (width 1) (layer "B.Cu") (net 2))
   (segment (start 208 88) (end 208 82) (width 1) (layer "B.Cu") (net 2))
@@
   (segment (start 168.499511 90.299511) (end 168.499511 130.600489) (width 1) (layer "B.Cu") (net 2))
   (segment (start 168.499511 130.600489) (end 162.1 137) (width 1) (layer "B.Cu") (net 2))
+  (segment (start 213.36 61.36) (end 208 61.36) (width 1) (layer "B.Cu") (net 2))
   (segment (start 61.4 141.7) (end 61.4 146.6) (width 1) (layer "B.Cu") (net 2))
   (segment (start 74.675 58.875) (end 75.325 58.875) (width 1) (layer "B.Cu") (net 2))
   (segment (start 63.6 139.5) (end 61.4 141.7) (width 1) (layer "B.Cu") (net 2))
+  (segment (start 208 76.6) (end 212.4 76.6) (width 1) (layer "B.Cu") (net 2))
   (segment (start 56 143) (end 56 147) (width 1) (layer "B.Cu") (net 2))
   (segment (start 56.14 62.16) (end 56.14 137.14) (width 1) (layer "B.Cu") (net 2))
+  (segment (start 215 63) (end 213.36 61.36) (width 1) (layer "B.Cu") (net 2))
   (segment (start 164.1 139.5) (end 63.6 139.5) (width 1) (layer "B.Cu") (net 2))
   (segment (start 75.325 58.875) (end 76.4 57.8) (width 1) (layer "B.Cu") (net 2))
@@
   (segment (start 179.225 91.655) (end 174.645 91.655) (width 1) (layer "B.Cu") (net 2))
   (segment (start 89.365 56.335) (end 89.915 56.335) (width 1) (layer "B.Cu") (net 2))
+  (segment (start 215 74) (end 215 63) (width 1) (layer "B.Cu") (net 2))
   (segment (start 87.9 57.8) (end 89.365 56.335) (width 1) (layer "B.Cu") (net 2))
   (segment (start 56.14 137.14) (end 59 140) (width 1) (layer "B.Cu") (net 2))
@@
   (segment (start 224 51) (end 216.58 43.58) (width 0.5) (layer "B.Cu") (net 47))
   (segment (start 216.58 43.58) (end 208 43.58) (width 0.5) (layer "B.Cu") (net 47))
-  (segment (start 215.9 78) (end 220.9 73) (width 0.8) (layer "B.Cu") (net 48))
-  (segment (start 145.1 71.6) (end 151.5 78) (width 0.8) (layer "B.Cu") (net 48))
+  (segment (start 145.1 71.6) (end 152.5 79) (width 0.8) (layer "B.Cu") (net 48))
+  (segment (start 220.9 73) (end 220.9 50.6) (width 0.8) (layer "B.Cu") (net 48))
+  (segment (start 216.42 46.12) (end 208 46.12) (width 0.8) (layer "B.Cu") (net 48))
   (segment (start 145.1 57.2) (end 145.1 71.6) (width 0.8) (layer "B.Cu") (net 48))
+  (segment (start 150.86 53.83) (end 148.47 53.83) (width 0.8) (layer "B.Cu") (net 48))
+  (segment (start 148.47 53.83) (end 145.1 57.2) (width 0.8) (layer "B.Cu") (net 48))
+  (segment (start 152.5 79) (end 214.9 79) (width 0.8) (layer "B.Cu") (net 48))
   (segment (start 220.9 50.6) (end 216.42 46.12) (width 0.8) (layer "B.Cu") (net 48))
-  (segment (start 216.42 46.12) (end 208 46.12) (width 0.8) (layer "B.Cu") (net 48))
-  (segment (start 151.5 78) (end 215.9 78) (width 0.8) (layer "B.Cu") (net 48))
-  (segment (start 220.9 73) (end 220.9 50.6) (width 0.8) (layer "B.Cu") (net 48))
-  (segment (start 148.47 53.83) (end 145.1 57.2) (width 0.8) (layer "B.Cu") (net 48))
-  (segment (start 150.86 53.83) (end 148.47 53.83) (width 0.8) (layer "B.Cu") (net 48))
+  (segment (start 214.9 79) (end 220.9 73) (width 0.8) (layer "B.Cu") (net 48))
   (segment (start 200 75) (end 199 76) (width 0.8) (layer "F.Cu") (net 49))
   (segment (start 200 53) (end 200 75) (width 0.8) (layer "F.Cu") (net 49))
